Commit message: corrected the limit float notation

File: xarm_description/urdf/lite6.urdf (robot description, URDF)
Before this commit: robot lite6_urdf, 8 links, 7 joints
Joints:
- joint joint1: limit lower=${-2.0*pi} upper={2.0*pi} effort=32 velocity=3.14 -> lower=-6.28319 upper=6.28319 effort=32 velocity=3.14
- joint joint2: limit lower=${-2.61799} upper=${2.61799} effort=32 velocity=3.14 -> lower=-2.61799 upper=2.61799 effort=32 velocity=3.14
- joint joint3: limit lower=${-0.061087} upper=${5.235988} effort=18 velocity=3.14 -> lower=-0.061087 upper=5.235988 effort=18 velocity=3.14
- joint joint4: limit lower=${-2.0*pi} upper=${2.0*pi} effort=2.5 velocity=3.14 -> lower=-6.28319 upper=6.28319 effort=2.5 velocity=3.14
- joint joint5: limit lower=${-2.1642} upper=${2.1642} effort=2.5 velocity=3.14 -> lower=-2.1642 upper=2.1642 effort=2.5 velocity=3.14
- joint joint6: limit lower=${-2.0*pi} upper=${2.0*pi} effort=2.5 velocity=3.14 -> lower=-6.28319 upper=6.28319 effort=2.5 velocity=3.14

Commit message: correct the mesh link for base

File: xarm_description/urdf/lite6.urdf (robot description, URDF)
Before this commit: robot lite6_urdf, 8 links, 7 joints
Links:
- link link_base: geometry collision mesh filename=package://xarm_description/meshes/lite6/collision/base_link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; visual mesh filename=package://xarm_description/meshes/lite6/visual/base.stl

Commit message: added urdf file provided by ufactory team

File: xarm_description/urdf/lite6.urdf (robot description, URDF)
Before this commit: robot lite6_urdf, 8 links, 7 joints
Links:
- removed link base
- removed link link_6
- added link link6, mass 0.180; collision mesh filename=package://xarm_description/meshes/lite6/collision/link6.stl; visual mesh filename=package://xarm_description/meshes/lite6/visual/link6.stl
- added link link_eef
- link link1: mass None -> 1.411
- link link2: mass None -> 1.34
- link link3: mass None -> 0.953
- link link4: mass None -> 1.284
- link link5: mass None -> 0.804
- link link_base: mass None -> 2.11; geometry collision mesh filename=package://xarm_description/meshes/lite6/collision/base.stl; visual mesh filename=package://xarm_description/meshes/lite6/visual/base.stl
Joints:
- removed joint base_link-base
- added joint joint_eef: type fixed, parent link6, child link_eef, origin xyz=0 0 0 rpy=0 0 0
- joint joint1: child link_1 -> link1; limit lower=-6.28319 upper=6.28319 effort=32 velocity=3.14 -> lower=-6.28 upper=6.28 effort=32.0 velocity=3.14
- joint joint2: limit lower=-2.61799 upper=2.61799 effort=32 velocity=3.14 -> lower=-2.61799 upper=2.61799 effort=32.0 velocity=3.14
- joint joint3: axis 0 1 0 -> 0 0 1; limit lower=-0.061087 upper=5.235988 effort=18 velocity=3.14 -> lower=-0.061087 upper=5.235988 effort=18.0 velocity=3.14
- joint joint4: limit lower=-6.28319 upper=6.28319 effort=2.5 velocity=3.14 -> lower=-6.28 upper=6.28 effort=2.5 velocity=3.14
- joint joint5: origin xyz=0 0 0  rpy=1.5708 0 0 -> xyz=0 0 0 rpy=1.5708 0 0
- joint joint6: limit lower=-6.28319 upper=6.28319 effort=2.5 velocity=3.14 -> lower=-6.28 upper=6.28 effort=2.5 velocity=3.14; origin xyz=0 0.0615 0  rpy=-1.5708 0 0 -> xyz=0 0.0615 0 rpy=-1.5708 0 0
